Commit message: did some renames on the aero_description packages #62

File: aero_arm_description/urdf/aero_arm.urdf.xacro (robot description, xacro)
@@ -1,58 +1,63 @@
-<robot name="AERO_arm" >
-  <link
-    name="base_link">
-    <inertial>
-      <origin
-        xyz="0 0 0"
-        rpy="0 0 0" />
-      <mass
-        value="0" />
+<robot xmlns:xacro="http://ros.org/wiki/xacro">
+<xacro:macro name="aero_arm" params="parent *origin prefix">
+   <joint name="arm_fixture" type="fixed">
+      <insert_block name="origin" />
+      <parent link="${parent}"/>
+      <child link="${prefix}_base_link"/>
+    </joint>
+  <link name="${prefix}_base_link">
+    <inertial>
+      <origin
+        xyz="0 0 0"
+        rpy="0 0 0" />
+      <mass
+        value="0.001" />
       <inertia
-        ixx="0"
-        ixy="0"
-        ixz="0"
-        iyy="0"
-        iyz="0"
-        izz="0" />
-    </inertial>
-    <visual>
-      <origin
-        xyz="0 0 0"
-        rpy="0 0 0" />
-      <geometry>
-        <mesh
-          filename="package://AERO_arm/meshes/base_link.STL" />
-      </geometry>
-      <material
-        name="">
-        <color
-          rgba="0.792156862745098 0.819607843137255 0.933333333333333 1" />
-      </material>
-    </visual>
-    <collision>
-      <origin
-        xyz="0 0 0"
-        rpy="0 0 0" />
-      <geometry>
-        <mesh
-          filename="package://AERO_arm/meshes/base_link.STL" />
-      </geometry>
-    </collision>
-  </link>
-  <link
-    name="Link1">
-    <inertial>
-      <origin
-        xyz="0 0 0"
-        rpy="0 0 0" />
-      <mass
-        value="0" />
-      <inertia
-        ixx="0"
-        ixy="0"
-        ixz="0"
-        iyy="0"
-        iyz="0"
-        izz="0" />
+        ixx="0.001"
+        ixy="0.001"
+        ixz="0.001"
+        iyy="0.001"
+        iyz="0.001"
+        izz="0.001" />
+    </inertial>
+    <visual>
+      <origin
+        xyz="0 0 0"
+        rpy="0 0 0" />
+      <geometry>
+        <mesh
+          filename="package://aero_arm/meshes/base_link.STL" />
+      </geometry>
+      <material
+        name="">
+        <color
+          rgba="0.792156862745098 0.819607843137255 0.933333333333333 1" />
+      </material>
+    </visual>
+    <collision>
+      <origin
+        xyz="0 0 0"
+        rpy="0 0 0" />
+      <geometry>
+        <mesh
+          filename="package://aero_arm/meshes/base_link.STL" />
+      </geometry>
+    </collision>
+  </link>
+  <link
+    name="${prefix}_Link1">
+    <inertial>
+      <origin
+        xyz="0 0 0"
+        rpy="0 0 0" />
+      <mass
+        value="0.001" />
+   <inertia
+        ixx="0.001"
+        ixy="0.001"
+        ixz="0.001"
+        iyy="0.001"
+        iyz="0.001"
+        izz="0.001" />
     </inertial>
     <visual>
@@ -62,5 +67,5 @@
       <geometry>
         <mesh
-          filename="package://AERO_arm/meshes/Link1.STL" />
+          filename="package://aero_arm/meshes/Link1.STL" />
       </geometry>
       <material
@@ -76,10 +81,10 @@
       <geometry>
         <mesh
-          filename="package://AERO_arm/meshes/Link1.STL" />
-      </geometry>
-    </collision>
-  </link>
-  <joint
-    name="Joint1"
+          filename="package://aero_arm/meshes/Link1.STL" />
+      </geometry>
+    </collision>
+  </link>
+  <joint
+    name="${prefix}_Joint1"
     type="continuous">
     <origin
@@ -87,25 +92,25 @@
       rpy="0 0 0" />
     <parent
-      link="base_link" />
-    <child
-      link="Link1" />
+      link="${prefix}_base_link" />
+    <child
+      link="${prefix}_Link1" />
     <axis
       xyz="0 0 -1" />
   </joint>
   <link
-    name="Link2">
-    <inertial>
-      <origin
-        xyz="0 0 0"
-        rpy="0 0 0" />
-      <mass
-        value="0" />
-      <inertia
-        ixx="0"
-        ixy="0"
-        ixz="0"
-        iyy="0"
-        iyz="0"
-        izz="0" />
+    name="${prefix}_Link2">
+    <inertial>
+      <origin
+        xyz="0 0 0"
+        rpy="0 0 0" />
+      <mass
+        value="0.001" />
+    <inertia
+        ixx="0.001"
+        ixy="0.001"
+        ixz="0.001"
+        iyy="0.001"
+        iyz="0.001"
+        izz="0.001" />
     </inertial>
     <visual>
@@ -115,5 +120,5 @@
       <geometry>
         <mesh
-          filename="package://AERO_arm/meshes/Link2.STL" />
+          filename="package://aero_arm/meshes/Link2.STL" />
       </geometry>
       <material
@@ -129,10 +134,10 @@
       <geometry>
         <mesh
-          filename="package://AERO_arm/meshes/Link2.STL" />
-      </geometry>
-    </collision>
-  </link>
-  <joint
-    name="Joint2"
+          filename="package://aero_arm/meshes/Link2.STL" />
+      </geometry>
+    </collision>
+  </link>
+  <joint
+    name="${prefix}_Joint2"
     type="continuous">
    <!-- <origin
@@ -143,12 +148,12 @@
       rpy="0.0 -1.5708 0" />
     <parent
-      link="Link1" />
-    <child
-      link="Link2" />
+      link="${prefix}_Link1" />
+    <child
+      link="${prefix}_Link2" />
     <axis
       xyz="0 0 -1" />
   </joint>
   <link
-    name="Link3">
+    name="${prefix}_Link3">
     <inertial>
 <!--
@@ -161,39 +166,39 @@
         rpy="0.00 0 0" />
       <mass
-        value="0" />
-      <inertia
-        ixx="0"
-        ixy="0"
-        ixz="0"
-        iyy="0"
-        iyz="0"
-        izz="0" />
-    </inertial>
-    <visual>
-      <origin
-        xyz="0 0 0"
-        rpy="0 0 0" />
-      <geometry>
-        <mesh
-          filename="package://AERO_arm/meshes/Link4_origin.STL" scale="0.001 0.001 0.001"/>
-      </geometry>
-      <material
-        name="">
-        <color
-          rgba="0.792156862745098 0.819607843137255 0.933333333333333 1" />
-      </material>
-    </visual>
-    <collision>
-      <origin
-        xyz="0 0 0"
-        rpy="0 0 0" />
-      <geometry>
-        <mesh
-          filename="package://AERO_arm/meshes/Link4_origin.STL" scale="0.001 0.001 0.001"/>
-      </geometry>
-    </collision>
-  </link>
-  <joint
-    name="Joint3"
+        value="0.001" />
+  <inertia
+        ixx="0.001"
+        ixy="0.001"
+        ixz="0.001"
+        iyy="0.001"
+        iyz="0.001"
+        izz="0.001" />
+    </inertial>
+    <visual>
+      <origin
+        xyz="0 0 0"
+        rpy="0 0 0" />
+      <geometry>
+        <mesh
+          filename="package://aero_arm/meshes/Link4_origin.STL" scale="0.001 0.001 0.001"/>
+      </geometry>
+      <material
+        name="">
+        <color
+          rgba="0.792156862745098 0.819607843137255 0.933333333333333 1" />
+      </material>
+    </visual>
+    <collision>
+      <origin
+        xyz="0 0 0"
+        rpy="0 0 0" />
+      <geometry>
+        <mesh
+          filename="package://aero_arm/meshes/Link4_origin.STL" scale="0.001 0.001 0.001"/>
+      </geometry>
+    </collision>
+  </link>
+  <joint
+    name="${prefix}_Joint3"
     type="continuous">
 <!--
@@ -206,52 +211,52 @@
       rpy="-3.1416 0 -0.28747" />
     <parent
-      link="Link2" />
-    <child
-      link="Link3" />
+      link="${prefix}_Link2" />
+    <child
+      link="${prefix}_Link3" />
     <axis
       xyz="0 0 -1" />
   </joint>
   <link
-    name="Link4">
-    <inertial>
-      <origin
-        xyz="0 0 0"
-        rpy="0 0 0" />
-      <mass
-        value="0" />
-      <inertia
-        ixx="0"
-        ixy="0"
-        ixz="0"
-        iyy="0"
-        iyz="0"
-        izz="0" />
-    </inertial>
-    <visual>
-      <origin
-        xyz="0 0 0"
-        rpy="0 0 0" />
-      <geometry>
-        <mesh
-          filename="package://AERO_arm/meshes/origin_fixed.STL" scale="0.001 0.001 0.001"/>
-      </geometry>
-      <material
-        name="">
-        <color
-          rgba="0.792156862745098 0.819607843137255 0.933333333333333 1" />
-      </material>
-    </visual>
-    <collision>
-      <origin
-        xyz="0 0 0"
-        rpy="0 0 0" />
-      <geometry>
-        <mesh
-          filename="package://AERO_arm/meshes/origin_fixed.STL" scale="0.001 0.001 0.001"/>
-      </geometry>
-    </collision>
-  </link>
-  <joint
-    name="Joint4"
+    name="${prefix}_Link4">
+    <inertial>
+      <origin
+        xyz="0 0 0"
+        rpy="0 0 0" />
+      <mass
+        value="0.001" />
+ <inertia
+        ixx="0.001"
+        ixy="0.001"
+        ixz="0.001"
+        iyy="0.001"
+        iyz="0.001"
+        izz="0.001" />
+    </inertial>
+    <visual>
+      <origin
+        xyz="0 0 0"
+        rpy="0 0 0" />
+      <geometry>
+        <mesh
+          filename="package://aero_arm/meshes/origin_fixed.STL" scale="0.001 0.001 0.001"/>
+      </geometry>
+      <material
+        name="">
+        <color
+          rgba="0.792156862745098 0.819607843137255 0.933333333333333 1" />
+      </material>
+    </visual>
+    <collision>
+      <origin
+        xyz="0 0 0"
+        rpy="0 0 0" />
+      <geometry>
+        <mesh
+          filename="package://aero_arm/meshes/origin_fixed.STL" scale="0.001 0.001 0.001"/>
+      </geometry>
+    </collision>
+  </link>
+  <joint
+    name="${prefix}_Joint4"
     type="continuous">
 <!--
@@ -264,52 +269,52 @@
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
File: aero_description/urdf/aero.urdf.xacro (robot description, xacro)
@@ -39,12 +39,12 @@
     xmlns:renderable="http://playerstage.sourceforge.net/gazebo/xmlschema/#renderable"
     xmlns:physics="http://playerstage.sourceforge.net/gazebo/xmlschema/#physics"
-	xmlns:xacro="http://ros.org/wiki/xacro" name="AERO">
+	xmlns:xacro="http://ros.org/wiki/xacro" name="aero">
 	<!-- Included URDF/XACRO Files -->
     <include filename="$(find husky_description)/urdf/materials.urdf.xacro" />
     <include filename="$(find husky_description)/urdf/wheel.urdf.xacro" />
     <include filename="$(find husky_description)/urdf/parts.urdf.xacro" />
-    <include filename="$(find AERO_description)/urdf/manta_camera.urdf.xacro" />
-    <include filename="$(find AERO_description)/urdf/sick_laser.urdf.xacro" />
-    <include filename="$(find AERO_arm)/robots/AERO_arm.urdf.xacro" />
+    <include filename="$(find aero_description)/urdf/manta_camera.urdf.xacro" />
+    <include filename="$(find aero_description)/urdf/sick_laser.urdf.xacro" />
+    <include filename="$(find aero_arm_description)/urdf/aero_arm.urdf.xacro" />
 	<!-- PROPERTY LIST -->
     <!--All units in m-kg-s-radians unit system -->
@@ -199,6 +199,6 @@
     </gazebo>
    <!-- Kinova Arm -->
-   <xacro:AERO_arm parent="base_link_top_plate_part" prefix="arm">
+   <xacro:aero_arm parent="base_link_top_plate_part" prefix="arm">
 	<origin xyz="0.20 -0.12 0.38" rpy="0 0 0" />
-   </xacro:AERO_arm>
+   </xacro:aero_arm>
 </robot>

File: aero_description/urdf/manta_camera.urdf.xacro (robot description, xacro)
@@ -4,5 +4,5 @@
       xmlns:interface="http://playerstage.sourceforge.net/gazebo/xmlschema/#interface"
       xmlns:xacro="http://ros.org/wiki/xacro">
-  <include filename="$(find AERO_description)/urdf/manta_camera.gazebo.xacro" />
+  <include filename="$(find aero_description)/urdf/manta_camera.gazebo.xacro" />
   <xacro:macro name="manta_cam_v0" params="frame_name parent *origin camera_name">
     <joint name="${frame_name}_frame_joint" type="fixed">
@@ -15,5 +15,5 @@
         <origin xyz="0.0 0.0 0" rpy="0 0 0"/>
         <geometry>
-          <mesh filename="package://AERO_description/meshes/Manta-Camera-Lense.STL" />
+          <mesh filename="package://aero_description/meshes/Manta-Camera-Lense.STL" />
         </geometry>
       </visual>
@@ -28,5 +28,5 @@
       <origin xyz="0 0 0" rpy="0 0 0" />
       <geometry>
-        <mesh filename="package://AERO_description/meshes/Manta-Camera-Lense.STL" />
+        <mesh filename="package://aero_description/meshes/Manta-Camera-Lense.STL" />
       </geometry>
     </collision>

File: aero_description/urdf/sick_laser.urdf.xacro (robot description, xacro)
@@ -4,5 +4,5 @@
        xmlns:interface="http://playerstage.sourceforge.net/gazebo/xmlschema/#interface"
        xmlns:xacro="http://ros.org/wiki/xacro">
-  <include filename="$(find AERO_description)/urdf/sick_laser.gazebo.xacro" />
+  <include filename="$(find aero_description)/urdf/sick_laser.gazebo.xacro" />
   <xacro:macro name="sick_laser_v0" params="name parent *origin ros_topic update_rate">
     <joint name="${name}_joint" type="fixed">
@@ -21,5 +21,5 @@
         <origin xyz="0.0 0.0 0" rpy="0 0 0"/>
         <geometry>
-          <mesh filename="package://AERO_description/meshes/LMS151.STL"/>
+          <mesh filename="package://aero_description/meshes/LMS151.STL"/>
         </geometry>
       </visual>
@@ -27,5 +27,5 @@
       <origin xyz="0 0 0" rpy="0 0 0" />
       <geometry>
-        <mesh filename="package://AERO_description/meshes/LMS151.STL"/>
+        <mesh filename="package://aero_description/meshes/LMS151.STL"/>
       </geometry>
     </collision>
