Commit message: removed arm from robot urdf #62

File: aero_description/urdf/aero.urdf.xacro (robot description, xacro)
@@ -46,5 +46,12 @@
     <include filename="$(find aero_description)/urdf/manta_camera.urdf.xacro" />
     <include filename="$(find aero_description)/urdf/sick_laser.urdf.xacro" />
-    <include filename="$(find aero_arm_description)/urdf/aero_arm.urdf.xacro" />
+    <xacro:macro name="static_transform" params="name parent xyz rpy">
+      <link name="${name}"/>
+      <joint name="joint_${name}" type="fixed">
+	<parent link="${parent}"/>
+	<child link="${name}"/>
+	<origin xyz="${xyz}" rpy="${rpy}" />
+      </joint>
+    </xacro:macro>
 	<!-- PROPERTY LIST -->
     <!--All units in m-kg-s-radians unit system -->
@@ -198,7 +205,4 @@
         <material>Gazebo/White</material>
     </gazebo>
-   <!-- Kinova Arm -->
-   <xacro:aero_arm parent="base_link_top_plate_part" prefix="arm">
-	<origin xyz="0.20 -0.12 0.38" rpy="0 0 0" />
-   </xacro:aero_arm>
+    <xacro:static_transform parent="base_link_top_plate_part" name="arm_base" xyz="0.20 -0.12 0.38" rpy="0 0 0"/>
 </robot>

Commit message: Formatted urdf files and added stereo camera frames #62

File: aero_description/urdf/aero.urdf.xacro (robot description, xacro)
@@ -40,169 +40,149 @@
     xmlns:physics="http://playerstage.sourceforge.net/gazebo/xmlschema/#physics"
 	xmlns:xacro="http://ros.org/wiki/xacro" name="aero">
-	<!-- Included URDF/XACRO Files -->
-    <include filename="$(find husky_description)/urdf/materials.urdf.xacro" />
-    <include filename="$(find husky_description)/urdf/wheel.urdf.xacro" />
-    <include filename="$(find husky_description)/urdf/parts.urdf.xacro" />
-    <include filename="$(find aero_description)/urdf/manta_camera.urdf.xacro" />
-    <include filename="$(find aero_description)/urdf/sick_laser.urdf.xacro" />
-    <xacro:macro name="static_transform" params="name parent xyz rpy">
-      <link name="${name}"/>
-      <joint name="joint_${name}" type="fixed">
-	<parent link="${parent}"/>
-	<child link="${name}"/>
-	<origin xyz="${xyz}" rpy="${rpy}" />
-      </joint>
-    </xacro:macro>
-	<!-- PROPERTY LIST -->
-    <!--All units in m-kg-s-radians unit system -->
-    <property name="M_PI" value="3.1415926535897931" />
-    <!-- Main Body-base-->
-    <!-- Location of com : center of mass -->
-    <property name="base_x_com" value="-0.08748000" />
-    <property name="base_y_com" value="-0.00085000" />
-    <property name="base_z_com" value="0.09947000" />
-    <!-- Size of the base-->
-    <property name="base_x_size" value="0.98740000" />
-    <property name="base_y_size" value="0.57090000" />
-    <property name="base_z_size" value="0.24750000" />
-    <!--Weight of the base-->
-    <property name="base_mass" value="33.45489000" /> <!-- in kg-->
-    <!--Inertial values for the base at center of mass, aligned with coordinate system. Units are kg*m^2-->
-    <property name="base_ixx_com_cs" value="0.60216370" />
-    <property name="base_ixy_com_cs" value="-0.02364198" />
-    <property name="base_ixz_com_cs" value="-0.11972132" />
-    <property name="base_iyy_com_cs" value="1.73859574" />
-    <property name="base_iyz_com_cs" value="-0.00154437" />
-    <property name="base_izz_com_cs" value="2.02955229" />
-<!-- BASE-FOOTPRINT -->
-    <!-- base_footprint is a fictitious link(frame) that is on the ground right below base_link origin, navigation stack depends on this frame -->
-    <link name="base_footprint">
-        <inertial>
-            <mass value="0.0001" />
-            <origin xyz="0 0 0" />
-            <inertia ixx="0.0001" ixy="0.0" ixz="0.0"
-                iyy="0.0001" iyz="0.0"
-                izz="0.0001" />
-        </inertial>
-        <visual>
-            <origin xyz="0 0 0" rpy="0 0 0" />
-            <geometry>
-                <box size="0.001 0.001 0.001" />
-            </geometry>
-        </visual>
-    </link>
-    <gazebo reference="base_footprint">
-        <material>Gazebo/Green</material>
-        <turnGravityOff>false</turnGravityOff>
-    </gazebo>
-    <joint name="base_footprint_joint" type="fixed">
-		<origin xyz="0 0 ${wheel_x_size/2 - base_z_origin_to_wheel_origin - base_z_origin_offset - base_z_origin_offset}" rpy="0 0 0" />
-        <parent link="base_footprint"/>
-        <child link="base_link" />
-    </joint>
-    <!-- BASE-LINK -->
-    <!--Actual body/chassis of the robot-->
-    <link name="base_link">
-        <inertial>
-            <mass value="${base_mass}" />
-            <!--This is the pose of the inertial reference frame, relative to the link reference frame. The origin of the inertial reference frame needs to be at the center of gravity. The axes of the inertial reference frame do not need to be aligned with the principal axes of the inertia.-->
-            <origin xyz="${base_x_com} ${base_y_com} ${base_z_com}" />
-            <!--The 3x3 rotational inertia matrix. Because the rotational inertia matrix is symmetric, only 6 above-diagonal elements of this matrix are specified here, using the attributes ixx, ixy, ixz, iyy, iyz, izz.-->
-            <inertia ixx="${base_ixx_com_cs}" ixy="${base_ixy_com_cs}" ixz="${base_ixz_com_cs}"
-                iyy="${base_iyy_com_cs}" iyz="${base_iyz_com_cs}" izz="${base_izz_com_cs}" />
-        </inertial>
-        <visual>
-            <origin xyz="0 0 ${base_z_origin_offset}" rpy="0 0 0" />
-            <geometry>
-                <mesh filename="package://husky_description/Media/models/base_link.stl" />
-            </geometry>
-            <material name="Black" />
-        </visual>
-		<collision>
-			<origin xyz="0 0 ${wheel_x_size/2 - base_z_origin_to_wheel_origin - 0.02}" rpy="0 0 0 " />
-			<geometry>
-				<box size = "${base_x_size+0.02} ${base_y_size} ${base_z_size + 0.02}"/> <!--making it slightly bigger in x and z direction-->
-			</geometry>
-		</collision>
-    </link>
-    <gazebo reference="base_link">
-        <material>Gazebo/FlatBlack</material>
-        <turnGravityOff>false</turnGravityOff>
-    </gazebo>
-    <!-- WHEEL macros -->
-	<husky_wheel fb="back" lr="left" parent="base_link" translateX="-1" translateY="1" flipY="-1"/>
-	<husky_wheel fb="back" lr="right" parent="base_link" translateX="-1" translateY="-1" flipY="-1"/>
-	<husky_wheel fb="front" lr="left" parent="base_link" translateX="1" translateY="1" flipY="-1"/>
-	<husky_wheel fb="front" lr="right" parent="base_link" translateX="1" translateY="-1" flipY="-1"/>
-    <!-- DECORATIONS -->
-    <!-- Top Plate -->
-    <husky_part parent="base_link" name="top_plate" mesh="top_plate"
-          colour="Yellow"
-          translateX="0.0" translateY="0.0" translateZ="0.005"
-          rotateX="0.0" rotateY="0.0" rotateZ="0.0"/>
-    <gazebo reference="base_link_top_plate_part">
-        <material>Gazebo/Yellow</material>
-    </gazebo>
-    <!-- User Rail -->
-    <husky_part parent="base_link" name="user_rail" mesh="user_rail"
-          colour="DarkGray"
-          translateX="0.272" translateY="0.0" translateZ="0.245"
-          rotateX="0.0" rotateY="0.0" rotateZ="0.0"/>
-    <gazebo reference="base_link_user_rail_part">
-        <material>Gazebo/Grey</material>
-    </gazebo>
-    <!-- Bumpers -->
-    <husky_part parent="base_link" name="front_bumper" mesh="bumper"
-          colour="DarkGray"
-          translateX="0.490" translateY="0.0" translateZ="0.091"
-          rotateX="0.0" rotateY="0.0" rotateZ="0.0"/>
-    <gazebo reference="base_link_front_bumper_part">
-        <material>Gazebo/FlatBlack</material>
-    </gazebo>
-    <husky_part parent="base_link" name="rear_bumper" mesh="bumper"
-          colour="DarkGray"
-          translateX="-0.48" translateY="0.0" translateZ="0.091"
-          rotateX="0.0" rotateY="0.0" rotateZ="3.14"/>
-    <gazebo reference="base_link_rear_bumper_part">
-        <material>Gazebo/FlatBlack</material>
-    </gazebo>
-    <gazebo>
-		<controller:husky_plugin name="husky_diff_controller" plugin="libhusky_description.so">
-		        <alwaysOn>true</alwaysOn>
-		        <updateRate>100.0</updateRate>
-		        <backLeftJoint>joint_back_left_wheel</backLeftJoint>
-		        <backRightJoint>joint_back_right_wheel</backRightJoint>
-		        <frontLeftJoint>joint_front_left_wheel</frontLeftJoint>
-		        <frontRightJoint>joint_front_right_wheel</frontRightJoint>
-		        <wheelSeparation>${base_y_size}</wheelSeparation>
-		        <wheelDiameter>${wheel_x_size}</wheelDiameter>
-		        <torque>35</torque>
-        </controller:husky_plugin>
-	</gazebo>
-   <!-- Ben ADDed -->
-   <!-- Note: calibraton needs to be done to determine the offsets -->
-   <!-- Front camera -->
-   <xacro:manta_cam_v0 frame_name="bot_stereo/left" parent="base_link_user_rail_part" camera_name="bot_stereo/left">
-	<origin xyz="0.0 0.04 0.04" rpy="0 0 0" />
-   </xacro:manta_cam_v0>
-   <xacro:manta_cam_v0 frame_name="bot_stereo/right" parent="base_link_user_rail_part" camera_name="bot_stereo/right">
-	<origin xyz="0.0 -0.04 0.04" rpy="0 0 0" />
-   </xacro:manta_cam_v0>
-  <gazebo reference="r_camera_frame">
-        <material>Gazebo/Red</material>
-    </gazebo>
-   <xacro:manta_cam_v0 frame_name="down_camera" parent="base_link_front_bumper_part" camera_name="down_camera">
-	<origin xyz="-0.05 0 -0.05" rpy="0 ${M_PI/2} 0" />
-   </xacro:manta_cam_v0>
-   <gazebo reference="down_camera_frame">
-        <material>Gazebo/Red</material>
-    </gazebo>
-   <!-- Laser -->
-   <xacro:sick_laser_v0 name="lms151_laser" parent="base_link_front_bumper_part" ros_topic="front_laser" update_rate="25" >
-	<origin xyz="-0.05 0 0.05" rpy="0 0 0" />
-   </xacro:sick_laser_v0>
-   <gazebo reference="lms151_laser_link">
-        <material>Gazebo/White</material>
-    </gazebo>
-    <xacro:static_transform parent="base_link_top_plate_part" name="arm_base" xyz="0.20 -0.12 0.38" rpy="0 0 0"/>
+  <!-- Included URDF/XACRO Files -->
+  <include filename="$(find husky_description)/urdf/materials.urdf.xacro" />
+  <include filename="$(find husky_description)/urdf/wheel.urdf.xacro" />
+  <include filename="$(find husky_description)/urdf/parts.urdf.xacro" />
+  <include filename="$(find aero_description)/urdf/stereo_camera_pair.urdf.xacro" />
+  <include filename="$(find aero_description)/urdf/sick_laser.urdf.xacro" />
+  <include filename="$(find aero_description)/urdf/simple_transform.urdf.xacro" />
+  <!-- PROPERTY LIST -->
+  <!--All units in m-kg-s-radians unit system -->
+  <property name="M_PI" value="3.1415926535897931" />
+  <!-- Main Body-base-->
+  <!-- Location of com : center of mass -->
+  <property name="base_x_com" value="-0.08748000" />
+  <property name="base_y_com" value="-0.00085000" />
+  <property name="base_z_com" value="0.09947000" />
+  <!-- Size of the base-->
+  <property name="base_x_size" value="0.98740000" />
+  <property name="base_y_size" value="0.57090000" />
+  <property name="base_z_size" value="0.24750000" />
+  <!--Weight of the base-->
+  <property name="base_mass" value="33.45489000" /> <!-- in kg-->
+  <!--Inertial values for the base at center of mass, aligned with coordinate system. Units are kg*m^2-->
+  <property name="base_ixx_com_cs" value="0.60216370" />
+  <property name="base_ixy_com_cs" value="-0.02364198" />
+  <property name="base_ixz_com_cs" value="-0.11972132" />
+  <property name="base_iyy_com_cs" value="1.73859574" />
+  <property name="base_iyz_com_cs" value="-0.00154437" />
+  <property name="base_izz_com_cs" value="2.02955229" />
+  <!-- BASE-FOOTPRINT -->
+  <!-- base_footprint is a fictitious link(frame) that is on the ground right below base_link origin, navigation stack depends on this frame -->
+  <link name="base_footprint">
+    <inertial>
+      <mass value="0.0001" />
+      <origin xyz="0 0 0" />
+      <inertia ixx="0.0001" ixy="0.0" ixz="0.0"
+	       iyy="0.0001" iyz="0.0"
+	       izz="0.0001" />
+    </inertial>
+    <visual>
+      <origin xyz="0 0 0" rpy="0 0 0" />
+      <geometry>
+	<box size="0.001 0.001 0.001" />
+      </geometry>
+    </visual>
+  </link>
+  <gazebo reference="base_footprint">
+    <material>Gazebo/Green</material>
+    <turnGravityOff>false</turnGravityOff>
+  </gazebo>
+  <joint name="base_link_joint" type="fixed">
+    <origin xyz="0 0 ${wheel_x_size/2 - base_z_origin_to_wheel_origin - base_z_origin_offset - base_z_origin_offset}" rpy="0 0 0" />
+    <parent link="base_footprint"/>
+    <child link="base_link" />
+  </joint>
+  <!-- BASE-LINK -->
+  <!--Actual body/chassis of the robot-->
+  <link name="base_link">
+    <inertial>
+      <mass value="${base_mass}" />
+      <!--This is the pose of the inertial reference frame, relative to the link reference frame. The origin of the inertial reference frame needs to be at the center of gravity. The axes of the inertial reference frame do not need to be aligned with the principal axes of the inertia.-->
+      <origin xyz="${base_x_com} ${base_y_com} ${base_z_com}" />
+      <!--The 3x3 rotational inertia matrix. Because the rotational inertia matrix is symmetric, only 6 above-diagonal elements of this matrix are specified here, using the attributes ixx, ixy, ixz, iyy, iyz, izz.-->
+      <inertia ixx="${base_ixx_com_cs}" ixy="${base_ixy_com_cs}" ixz="${base_ixz_com_cs}"
+	       iyy="${base_iyy_com_cs}" iyz="${base_iyz_com_cs}" izz="${base_izz_com_cs}" />
+    </inertial>
+    <visual>
+      <origin xyz="0 0 ${base_z_origin_offset}" rpy="0 0 0" />
+      <geometry>
+	<mesh filename="package://husky_description/Media/models/base_link.stl" />
+      </geometry>
+      <material name="Black" />
+    </visual>
+    <collision>
+      <origin xyz="0 0 ${wheel_x_size/2 - base_z_origin_to_wheel_origin - 0.02}" rpy="0 0 0 " />
+      <geometry>
+	<box size = "${base_x_size+0.02} ${base_y_size} ${base_z_size + 0.02}"/> <!--making it slightly bigger in x and z direction-->
+      </geometry>
+    </collision>
+  </link>
+  <gazebo reference="base_link">
+    <material>Gazebo/FlatBlack</material>
+    <turnGravityOff>false</turnGravityOff>
+  </gazebo>
+  <!-- WHEEL macros -->
+  <husky_wheel fb="back" lr="left" parent="base_link" translateX="-1" translateY="1" flipY="-1"/>
+  <husky_wheel fb="back" lr="right" parent="base_link" translateX="-1" translateY="-1" flipY="-1"/>
+  <husky_wheel fb="front" lr="left" parent="base_link" translateX="1" translateY="1" flipY="-1"/>
+  <husky_wheel fb="front" lr="right" parent="base_link" translateX="1" translateY="-1" flipY="-1"/>
+  <!-- DECORATIONS -->
+  <!-- Top Plate -->
+  <husky_part parent="base_link" name="top_plate" mesh="top_plate"
+	      colour="Yellow"
+	      translateX="0.0" translateY="0.0" translateZ="0.005"
+	      rotateX="0.0" rotateY="0.0" rotateZ="0.0"/>
+  <gazebo reference="base_link_top_plate_part">
+    <material>Gazebo/Yellow</material>
+  </gazebo>
+  <!-- User Rail -->
+  <husky_part parent="base_link" name="user_rail" mesh="user_rail"
+	      colour="DarkGray"
+	      translateX="0.272" translateY="0.0" translateZ="0.245"
+	      rotateX="0.0" rotateY="0.0" rotateZ="0.0"/>
+  <gazebo reference="base_link_user_rail_part">
+    <material>Gazebo/Grey</material>
+  </gazebo>
+  <!-- Bumpers -->
+  <husky_part parent="base_link" name="front_bumper" mesh="bumper"
+	      colour="DarkGray"
+	      translateX="0.490" translateY="0.0" translateZ="0.091"
+	      rotateX="0.0" rotateY="0.0" rotateZ="0.0"/>
+  <gazebo reference="base_link_front_bumper_part">
+    <material>Gazebo/FlatBlack</material>
+  </gazebo>
+  <husky_part parent="base_link" name="rear_bumper" mesh="bumper"
+	      colour="DarkGray"
+	      translateX="-0.48" translateY="0.0" translateZ="0.091"
+	      rotateX="0.0" rotateY="0.0" rotateZ="3.14"/>
+  <gazebo reference="base_link_rear_bumper_part">
+    <material>Gazebo/FlatBlack</material>
+  </gazebo>
+  <gazebo>
+    <controller:husky_plugin name="husky_diff_controller" plugin="libhusky_description.so">
+      <alwaysOn>true</alwaysOn>
+      <updateRate>100.0</updateRate>
+      <backLeftJoint>joint_back_left_wheel</backLeftJoint>
+      <backRightJoint>joint_back_right_wheel</backRightJoint>
+      <frontLeftJoint>joint_front_left_wheel</frontLeftJoint>
+      <frontRightJoint>joint_front_right_wheel</frontRightJoint>
+      <wheelSeparation>${base_y_size}</wheelSeparation>
+      <wheelDiameter>${wheel_x_size}</wheelDiameter>
+      <torque>35</torque>
+    </controller:husky_plugin>
+  </gazebo>
+  <!-- Cameras -->
+  <xacro:stereo_camera_pair parent="base_link_front_bumper_part" prefix="lower_stereo" xyz="0 0 0" rpy="0 0 0" camera_offset="0.04"/>
+  <xacro:stereo_camera_pair parent="camera_boom" prefix="upper_stereo" xyz="0 0 0" rpy="0 0 0" camera_offset="0.04"/>
+  <xacro:pan_transform parent="base_link_top_plate_part" name="camera_boom" xyz="0 0 0.5" rpy="0 0 0"/>
+  <!-- Laser -->
+  <xacro:sick_laser_v0 name="laser" parent="base_link_front_bumper_part" ros_topic="laser" update_rate="25" >
+    <origin xyz="-0.05 0 0.05" rpy="0 0 0" />
+  </xacro:sick_laser_v0>
+  <gazebo reference="laser">
+    <material>Gazebo/White</material>
+  </gazebo>
+  <!-- Arm -->
+  <xacro:static_transform parent="base_link_front_bumper_part" name="arm_base" xyz="0.20 -0.12 0.38" rpy="0 0 0"/>
 </robot>

File: aero_description/urdf/sick_laser.urdf.xacro (robot description, xacro)
@@ -10,7 +10,7 @@
       <insert_block name="origin" />
       <parent link="${parent}"/>
-      <child link="${name}_link"/>
+      <child link="${name}"/>
     </joint>
-    <link name="${name}_link" type="laser">
+    <link name="${name}" type="laser">
       <inertial>
         <mass value="0.001" />
