Commit message: More cleanup of aero_description #62

File: aero_description/urdf/aero.urdf.xacro (robot description, xacro)
@@ -1,29 +1,3 @@
 <?xml version="1.0"?>
-<!--
-Copyright (c) 2012, Siddhant Ahuja (Sid), Ryan Gariepy
-All rights reserved.
-Redistribution and use in source and binary forms, with or without
-modification, are permitted provided that the following conditions are met:
-    * Redistributions of source code must retain the above copyright
-      notice, this list of conditions and the following disclaimer.
-    * Redistributions in binary form must reproduce the above copyright
-      notice, this list of conditions and the following disclaimer in the
-      documentation and/or other materials provided with the distribution.
-    * Neither the name of Clearpath Robotics nor the
-      names of its contributors may be used to endorse or promote products
-      derived from this software without specific prior written permission.
-THIS SOFTWARE IS PROVIDED BY THE COPYRIGHT HOLDERS AND CONTRIBUTORS "AS IS" AND
-ANY EXPRESS OR IMPLIED WARRANTIES, INCLUDING, BUT NOT LIMITED TO, THE IMPLIED
-WARRANTIES OF MERCHANTABILITY AND FITNESS FOR A PARTICULAR PURPOSE ARE
-DISCLAIMED. IN NO EVENT SHALL THE COPYRIGHT HOLDERS BE LIABLE FOR ANY
-DIRECT, INDIRECT, INCIDENTAL, SPECIAL, EXEMPLARY, OR CONSEQUENTIAL DAMAGES
-(INCLUDING, BUT NOT LIMITED TO, PROCUREMENT OF SUBSTITUTE GOODS OR SERVICES;
-LOSS OF USE, DATA, OR PROFITS; OR BUSINESS INTERRUPTION) HOWEVER CAUSED AND
-ON ANY THEORY OF LIABILITY, WHETHER IN CONTRACT, STRICT LIABILITY, OR TORT
-(INCLUDING NEGLIGENCE OR OTHERWISE) ARISING IN ANY WAY OUT OF THE USE OF THIS
-SOFTWARE, EVEN IF ADVISED OF THE POSSIBILITY OF SUCH DAMAGE.
-This program contains the description of the robot base model for the Clearpath
-Husky A200
--->
 <robot
 	xmlns:xi="http://www.w3.org/2001/XInclude"
@@ -41,140 +15,13 @@
 	xmlns:xacro="http://ros.org/wiki/xacro" name="aero">
   <!-- Included URDF/XACRO Files -->
-  <include filename="$(find husky_description)/urdf/materials.urdf.xacro" />
-  <include filename="$(find husky_description)/urdf/wheel.urdf.xacro" />
-  <include filename="$(find husky_description)/urdf/parts.urdf.xacro" />
+  <include filename="$(find aero_description)/urdf/husky.urdf.xacro" />
   <include filename="$(find aero_description)/urdf/stereo_camera_pair.urdf.xacro" />
   <include filename="$(find aero_description)/urdf/sick_laser.urdf.xacro" />
   <include filename="$(find aero_description)/urdf/simple_transform.urdf.xacro" />
-  <!-- PROPERTY LIST -->
-  <!--All units in m-kg-s-radians unit system -->
-  <property name="M_PI" value="3.1415926535897931" />
-  <!-- Main Body-base-->
-  <!-- Location of com : center of mass -->
-  <property name="base_x_com" value="-0.08748000" />
-  <property name="base_y_com" value="-0.00085000" />
-  <property name="base_z_com" value="0.09947000" />
-  <!-- Size of the base-->
-  <property name="base_x_size" value="0.98740000" />
-  <property name="base_y_size" value="0.57090000" />
-  <property name="base_z_size" value="0.24750000" />
-  <!--Weight of the base-->
-  <property name="base_mass" value="33.45489000" /> <!-- in kg-->
-  <!--Inertial values for the base at center of mass, aligned with coordinate system. Units are kg*m^2-->
-  <property name="base_ixx_com_cs" value="0.60216370" />
-  <property name="base_ixy_com_cs" value="-0.02364198" />
-  <property name="base_ixz_com_cs" value="-0.11972132" />
-  <property name="base_iyy_com_cs" value="1.73859574" />
-  <property name="base_iyz_com_cs" value="-0.00154437" />
-  <property name="base_izz_com_cs" value="2.02955229" />
-  <!-- BASE-FOOTPRINT -->
-  <!-- base_footprint is a fictitious link(frame) that is on the ground right below base_link origin, navigation stack depends on this frame -->
-  <link name="base_footprint">
-    <inertial>
-      <mass value="0.0001" />
-      <origin xyz="0 0 0" />
-      <inertia ixx="0.0001" ixy="0.0" ixz="0.0"
-	       iyy="0.0001" iyz="0.0"
-	       izz="0.0001" />
-    </inertial>
-    <visual>
-      <origin xyz="0 0 0" rpy="0 0 0" />
-      <geometry>
-	<box size="0.001 0.001 0.001" />
-      </geometry>
-    </visual>
-  </link>
-  <gazebo reference="base_footprint">
-    <material>Gazebo/Green</material>
-    <turnGravityOff>false</turnGravityOff>
-  </gazebo>
-  <joint name="base_link_joint" type="fixed">
-    <origin xyz="0 0 ${wheel_x_size/2 - base_z_origin_to_wheel_origin - base_z_origin_offset - base_z_origin_offset}" rpy="0 0 0" />
-    <parent link="base_footprint"/>
-    <child link="base_link" />
-  </joint>
-  <!-- BASE-LINK -->
-  <!--Actual body/chassis of the robot-->
-  <link name="base_link">
-    <inertial>
-      <mass value="${base_mass}" />
-      <!--This is the pose of the inertial reference frame, relative to the link reference frame. The origin of the inertial reference frame needs to be at the center of gravity. The axes of the inertial reference frame do not need to be aligned with the principal axes of the inertia.-->
-      <origin xyz="${base_x_com} ${base_y_com} ${base_z_com}" />
-      <!--The 3x3 rotational inertia matrix. Because the rotational inertia matrix is symmetric, only 6 above-diagonal elements of this matrix are specified here, using the attributes ixx, ixy, ixz, iyy, iyz, izz.-->
-      <inertia ixx="${base_ixx_com_cs}" ixy="${base_ixy_com_cs}" ixz="${base_ixz_com_cs}"
-	       iyy="${base_iyy_com_cs}" iyz="${base_iyz_com_cs}" izz="${base_izz_com_cs}" />
-    </inertial>
-    <visual>
-      <origin xyz="0 0 ${base_z_origin_offset}" rpy="0 0 0" />
-      <geometry>
-	<mesh filename="package://husky_description/Media/models/base_link.stl" />
-      </geometry>
-      <material name="Black" />
-    </visual>
-    <collision>
-      <origin xyz="0 0 ${wheel_x_size/2 - base_z_origin_to_wheel_origin - 0.02}" rpy="0 0 0 " />
-      <geometry>
-	<box size = "${base_x_size+0.02} ${base_y_size} ${base_z_size + 0.02}"/> <!--making it slightly bigger in x and z direction-->
-      </geometry>
-    </collision>
-  </link>
-  <gazebo reference="base_link">
-    <material>Gazebo/FlatBlack</material>
-    <turnGravityOff>false</turnGravityOff>
-  </gazebo>
-  <!-- WHEEL macros -->
-  <husky_wheel fb="back" lr="left" parent="base_link" translateX="-1" translateY="1" flipY="-1"/>
-  <husky_wheel fb="back" lr="right" parent="base_link" translateX="-1" translateY="-1" flipY="-1"/>
-  <husky_wheel fb="front" lr="left" parent="base_link" translateX="1" translateY="1" flipY="-1"/>
-  <husky_wheel fb="front" lr="right" parent="base_link" translateX="1" translateY="-1" flipY="-1"/>
-  <!-- DECORATIONS -->
-  <!-- Top Plate -->
-  <husky_part parent="base_link" name="top_plate" mesh="top_plate"
-	      colour="Yellow"
-	      translateX="0.0" translateY="0.0" translateZ="0.005"
-	      rotateX="0.0" rotateY="0.0" rotateZ="0.0"/>
-  <gazebo reference="base_link_top_plate_part">
-    <material>Gazebo/Yellow</material>
-  </gazebo>
-  <!-- User Rail -->
-  <husky_part parent="base_link" name="user_rail" mesh="user_rail"
-	      colour="DarkGray"
-	      translateX="0.272" translateY="0.0" translateZ="0.245"
-	      rotateX="0.0" rotateY="0.0" rotateZ="0.0"/>
-  <gazebo reference="base_link_user_rail_part">
-    <material>Gazebo/Grey</material>
-  </gazebo>
-  <!-- Bumpers -->
-  <husky_part parent="base_link" name="front_bumper" mesh="bumper"
-	      colour="DarkGray"
-	      translateX="0.490" translateY="0.0" translateZ="0.091"
-	      rotateX="0.0" rotateY="0.0" rotateZ="0.0"/>
-  <gazebo reference="base_link_front_bumper_part">
-    <material>Gazebo/FlatBlack</material>
-  </gazebo>
-  <husky_part parent="base_link" name="rear_bumper" mesh="bumper"
-	      colour="DarkGray"
-	      translateX="-0.48" translateY="0.0" translateZ="0.091"
-	      rotateX="0.0" rotateY="0.0" rotateZ="3.14"/>
-  <gazebo reference="base_link_rear_bumper_part">
-    <material>Gazebo/FlatBlack</material>
-  </gazebo>
-  <gazebo>
-    <controller:husky_plugin name="husky_diff_controller" plugin="libhusky_description.so">
-      <alwaysOn>true</alwaysOn>
-      <updateRate>100.0</updateRate>
-      <backLeftJoint>joint_back_left_wheel</backLeftJoint>
-      <backRightJoint>joint_back_right_wheel</backRightJoint>
-      <frontLeftJoint>joint_front_left_wheel</frontLeftJoint>
-      <frontRightJoint>joint_front_right_wheel</frontRightJoint>
-      <wheelSeparation>${base_y_size}</wheelSeparation>
-      <wheelDiameter>${wheel_x_size}</wheelDiameter>
-      <torque>35</torque>
-    </controller:husky_plugin>
-  </gazebo>
+  <xacro:husky/>
   <!-- Cameras -->
-  <xacro:stereo_camera_pair parent="base_link_front_bumper_part" prefix="lower_stereo" xyz="0 0 0" rpy="0 0 0" camera_offset="0.04"/>
-  <xacro:stereo_camera_pair parent="camera_boom" prefix="upper_stereo" xyz="0 0 0" rpy="0 0 0" camera_offset="0.04"/>
-  <xacro:pan_transform parent="base_link_top_plate_part" name="camera_boom" xyz="0 0 0.5" rpy="0 0 0"/>
+  <xacro:stereo_camera_pair parent="base_link_front_bumper_part" prefix="lower_stereo" xyz="0.02 0 0.02" rpy="0 0.2 0" camera_offset="0.04"/>
+  <xacro:stereo_camera_pair parent="camera_boom" prefix="upper_stereo" xyz="0.02 0 0.02" rpy="0 0.2 0" camera_offset="0.04"/>
+  <xacro:revolute_pan_transform parent="base_link_top_plate_part" name="camera_boom" xyz="0 0 0.9" rpy="0 0 0" lower_limit="-2" upper_limit="2"/>
   <!-- Laser -->
   <xacro:sick_laser_v0 name="laser" parent="base_link_front_bumper_part" ros_topic="laser" update_rate="25" >
@@ -185,4 +32,4 @@
   </gazebo>
   <!-- Arm -->
-  <xacro:static_transform parent="base_link_front_bumper_part" name="arm_base" xyz="0.20 -0.12 0.38" rpy="0 0 0"/>
+  <xacro:static_transform parent="base_link_front_bumper_part" name="arm_base" xyz="0.20 0 0.38" rpy="0 0 0"/>
 </robot>

File: aero_description/urdf/simple_transform.urdf.xacro (robot description, xacro)
@@ -12,5 +12,5 @@
       </joint>
     </xacro:macro>
-    <xacro:macro name="pan_transform" params="name parent xyz rpy">
+    <xacro:macro name="continuouspan_transform" params="name parent xyz rpy">
       <link name="${name}"/>
       <joint name="${name}_joint" type="continuous">
@@ -21,3 +21,13 @@
       </joint>
     </xacro:macro>
+    <xacro:macro name="revolute_pan_transform" params="name parent xyz rpy lower_limit upper_limit">
+      <link name="${name}"/>
+      <joint name="${name}_joint" type="revolute">
+	<parent link="${parent}"/>
+	<child link="${name}"/>
+	<origin xyz="${xyz}" rpy="${rpy}" />
+	<axis xyz="0 0 1"/>
+	<limit lower="${lower_limit}" upper="${upper_limit}" effort="1000" velocity="6"/>
+      </joint>
+    </xacro:macro>
 </root>

Commit message: improved urdf model #62

File: aero_description/urdf/aero.urdf.xacro (robot description, xacro)
@@ -21,10 +21,18 @@
   <xacro:husky/>
   <!-- Cameras -->
-  <xacro:stereo_camera_pair parent="base_link_front_bumper_part" prefix="lower_stereo" xyz="0.02 0 0.02" rpy="0 0.2 0" camera_offset="0.04"/>
-  <xacro:stereo_camera_pair parent="camera_boom" prefix="upper_stereo" xyz="0.02 0 0.02" rpy="0 0.2 0" camera_offset="0.04"/>
-  <xacro:revolute_pan_transform parent="base_link_top_plate_part" name="camera_boom" xyz="0 0 0.9" rpy="0 0 0" lower_limit="-2" upper_limit="2"/>
+  <xacro:stereo_camera_pair parent="base_link_front_bumper_part" prefix="lower_stereo" xyz="0.07 0 0.02" rpy="0 0.2 0" camera_offset="0.08"/>
+  <xacro:stereo_camera_pair parent="camera_boom" prefix="upper_stereo" xyz="0.02 0 0.02" rpy="0 0.2 0" camera_offset="0.08"/>
+  <xacro:revolute_pan_transform parent="base_link_top_plate_part" name="camera_boom" xyz="0 0 0.9" rpy="0 0 0" lower_limit="-2" upper_limit="2">
+    <visual>
+      <origin xyz="0.0 0.0 -0.45" rpy="0 0 0" />
+      <geometry>
+	<cylinder length="0.9" radius="0.01" />
+      </geometry>
+      <material name="DarkGray" />
+    </visual>
+  </xacro:revolute_pan_transform>
   <!-- Laser -->
   <xacro:sick_laser_v0 name="laser" parent="base_link_front_bumper_part" ros_topic="laser" update_rate="25" >
-    <origin xyz="-0.05 0 0.05" rpy="0 0 0" />
+    <origin xyz="0.03 0 0.05" rpy="0 0 0" />
   </xacro:sick_laser_v0>
   <gazebo reference="laser">
@@ -32,4 +40,12 @@
   </gazebo>
   <!-- Arm -->
-  <xacro:static_transform parent="base_link_front_bumper_part" name="arm_base" xyz="0.20 0 0.38" rpy="0 0 0"/>
+  <xacro:static_transform parent="base_link_front_bumper_part" name="arm_base" xyz="-0.04 0 -0.03" rpy="0 0 0">
+    <visual>
+      <origin xyz="0 0 0" rpy="0 0 0" />
+      <geometry>
+	<box size="0.01 0.01 0.01" />
+      </geometry>
+      <material name="Blue" />
+    </visual>
+  </xacro:static_transform>
 </robot>

File: aero_description/urdf/husky.urdf.xacro (robot description, xacro)
@@ -42,6 +42,6 @@
   <!-- Included URDF/XACRO Files -->
   <include filename="$(find husky_description)/urdf/materials.urdf.xacro" />
-  <include filename="$(find husky_description)/urdf/wheel.urdf.xacro" />
-  <include filename="$(find husky_description)/urdf/parts.urdf.xacro" />
+  <include filename="$(find aero_description)/urdf/wheel.urdf.xacro" />
+  <include filename="$(find aero_description)/urdf/parts.urdf.xacro" />
   <!-- PROPERTY LIST -->
   <!--All units in m-kg-s-radians unit system -->
@@ -104,7 +104,11 @@
       </inertial>
       <visual>
-	<origin xyz="0 0 ${base_z_origin_offset}" rpy="0 0 0" />
+<!--	<origin xyz="0 0 ${base_z_origin_offset}" rpy="0 0 0" />
 	<geometry>
 	  <mesh filename="package://husky_description/Media/models/base_link.stl" />
+	</geometry>-->
+	<origin xyz="0 0 ${wheel_x_size/2 - base_z_origin_to_wheel_origin - 0.02}" rpy="0 0 0 " />
+	<geometry>
+	  <box size = "${base_x_size+0.02} ${base_y_size} ${base_z_size + 0.02}"/> <!--making it slightly bigger in x and z direction-->
 	</geometry>
 	<material name="Black" />

File: aero_description/urdf/simple_transform.urdf.xacro (robot description, xacro)
@@ -4,6 +4,8 @@
       xmlns:interface="http://playerstage.sourceforge.net/gazebo/xmlschema/#interface"
       xmlns:xacro="http://ros.org/wiki/xacro">
-    <xacro:macro name="static_transform" params="name parent xyz rpy">
-      <link name="${name}"/>
+    <xacro:macro name="static_transform" params="name parent xyz rpy *visual">
+      <link name="${name}">
+	<xacro:insert_block name="visual" />
+      </link>
       <joint name="${name}_joint" type="fixed">
 	<parent link="${parent}"/>
@@ -12,6 +14,8 @@
       </joint>
     </xacro:macro>
-    <xacro:macro name="continuouspan_transform" params="name parent xyz rpy">
-      <link name="${name}"/>
+    <xacro:macro name="continuouspan_transform" params="name parent xyz rpy *visual">
+      <link name="${name}">
+	<xacro:insert_block name="visual" />
+      </link>
       <joint name="${name}_joint" type="continuous">
 	<parent link="${parent}"/>
@@ -21,6 +25,8 @@
       </joint>
     </xacro:macro>
-    <xacro:macro name="revolute_pan_transform" params="name parent xyz rpy lower_limit upper_limit">
-      <link name="${name}"/>
+    <xacro:macro name="revolute_pan_transform" params="name parent xyz rpy lower_limit upper_limit *visual">
+      <link name="${name}">
+	<xacro:insert_block name="visual" />
+      </link>
       <joint name="${name}_joint" type="revolute">
 	<parent link="${parent}"/>

File: aero_description/urdf/stereo_camera_pair.urdf.xacro (robot description, xacro)
@@ -7,10 +7,13 @@
   <include filename="$(find aero_description)/urdf/manta_camera.urdf.xacro" />
   <xacro:macro name="stereo_camera_pair" params="prefix parent xyz rpy camera_offset">
-    <link name="${prefix}/camera_rail"/>
-    <joint name="${prefix}/joint_camera_rail" type="fixed">
-      <parent link="${parent}"/>
-      <child link="${prefix}/camera_rail"/>
-      <origin xyz="${xyz}" rpy="${rpy}" />
-    </joint>
+    <xacro:static_transform parent="${parent}" name="${prefix}/camera_rail" xyz="${xyz}" rpy="${rpy}">
+    <visual>
+      <origin xyz="-0.03 0 -0.018" rpy="0 0 0" />
+      <geometry>
+	<box size="0.05 ${camera_offset+0.04} 0.013" />
+      </geometry>
+      <material name="Red"/>
+    </visual>
+  </xacro:static_transform>
     <xacro:manta_cam_v0 frame_name="${prefix}/left_camera" parent="${prefix}/camera_rail" camera_name="${prefix}/left">
       <origin xyz="0.0 ${camera_offset/2} 0.0" rpy="0 0 0" />
@@ -19,5 +22,14 @@
       <origin xyz="0.0 ${-camera_offset/2} 0.0" rpy="0 0 0" />
     </xacro:manta_cam_v0>
-    <xacro:static_transform parent="${prefix}/camera_rail" name="${prefix}/optical_frame" xyz="0 0 0" rpy="0 0 0"/>
+    <xacro:static_transform parent="${prefix}/camera_rail" name="${prefix}/optical_frame" xyz="0 0 0" rpy="0 0 0">
+    <visual>
+      <geometry>
+	<box size="0 0 0" />
+      </geometry>
+      <material name="Clear">
+	<color rgba="0 0 0 0"/>
+      </material>
+    </visual>
+  </xacro:static_transform>
   </xacro:macro>
 </root>

Commit message: Integrated urdf into aero_base #62 drive controller now publishes joint position

File: aero_description/urdf/aero.urdf.xacro (robot description, xacro)
@@ -22,10 +22,10 @@
   <!-- Cameras -->
   <xacro:stereo_camera_pair parent="base_link_front_bumper_part" prefix="lower_stereo" xyz="0.07 0 0.02" rpy="0 0.2 0" camera_offset="0.08"/>
-  <xacro:stereo_camera_pair parent="camera_boom" prefix="upper_stereo" xyz="0.02 0 0.02" rpy="0 0.2 0" camera_offset="0.08"/>
-  <xacro:revolute_pan_transform parent="base_link_top_plate_part" name="camera_boom" xyz="0 0 0.9" rpy="0 0 0" lower_limit="-2" upper_limit="2">
+  <xacro:stereo_camera_pair parent="boom" prefix="upper_stereo" xyz="0.02 0 0.02" rpy="0 0.2 0" camera_offset="0.08"/>
+  <xacro:revolute_pan_transform parent="base_link_top_plate_part" name="boom" xyz="0 0 0.9" rpy="0 0 0" lower_limit="-2" upper_limit="2">
     <visual>
       <origin xyz="0.0 0.0 -0.45" rpy="0 0 0" />
       <geometry>
-	<cylinder length="0.9" radius="0.01" />
+	<cylinder length="0.9" radius="0.02" />
       </geometry>
       <material name="DarkGray" />
@@ -33,8 +33,8 @@
   </xacro:revolute_pan_transform>
   <!-- Laser -->
-  <xacro:sick_laser_v0 name="laser" parent="base_link_front_bumper_part" ros_topic="laser" update_rate="25" >
+  <xacro:sick_laser_v0 name="lidar" parent="base_link_front_bumper_part" ros_topic="laser" update_rate="25" >
     <origin xyz="0.03 0 0.05" rpy="0 0 0" />
   </xacro:sick_laser_v0>
-  <gazebo reference="laser">
+  <gazebo reference="lidar">
     <material>Gazebo/White</material>
   </gazebo>
@@ -49,3 +49,13 @@
     </visual>
   </xacro:static_transform>
+  <!-- IMU -->
+  <xacro:static_transform parent="base_link" name="imu" xyz="0.06 0 0" rpy="0 0 0">
+    <visual>
+      <origin xyz="0 0 0" rpy="0 0 0" />
+      <geometry>
+	<box size="0.01 0.01 0.01" />
+      </geometry>
+      <material name="Blue" />
+    </visual>
+  </xacro:static_transform>
 </robot>
