Commit message: Updated urdf with CAD measurements #62

File: aero_description/urdf/aero.urdf.xacro (robot description, xacro)
@@ -21,7 +21,16 @@
   <xacro:husky/>
   <!-- Cameras -->
-  <xacro:stereo_camera_pair parent="base_link_front_bumper_part" prefix="lower_stereo" xyz="0.07 0 0.02" rpy="0 0.2 0" camera_offset="0.08"/>
-  <xacro:stereo_camera_pair parent="boom" prefix="upper_stereo" xyz="0.02 0 0.02" rpy="0 0.2 0" camera_offset="0.08"/>
-  <xacro:revolute_pan_transform parent="base_link_top_plate_part" name="boom" xyz="0 0 0.9" rpy="0 0 0" lower_limit="-2" upper_limit="2">
+  <xacro:stereo_camera_pair parent="base_link_front_mount_part" prefix="lower_stereo" xyz="0.07 0 0.02" rpy="0 0.2 0" camera_offset="0.08"/>
+  <xacro:stereo_camera_pair parent="boom" prefix="upper_stereo" xyz="0 0 0.022606" rpy="0 0.2 0" camera_offset="0.294386"/>
+  <xacro:static_transform parent="base_link_top_plate_part" name="boom_base" xyz="-0.422402 0 -0.09906" rpy="0 0 0">
+    <visual>
+      <origin xyz="0 0 0" rpy="0 0 0" />
+      <geometry>
+	<box size="0.01 0.01 0.01" />
+      </geometry>
+      <material name="Blue" />
+    </visual>
+  </xacro:static_transform>
+  <xacro:revolute_pan_transform parent="boom_base" name="boom" xyz="0 0 1.014476" rpy="0 0 0" lower_limit="-2" upper_limit="2">
     <visual>
       <origin xyz="0.0 0.0 -0.45" rpy="0 0 0" />
@@ -33,6 +42,6 @@
   </xacro:revolute_pan_transform>
   <!-- Laser -->
-  <xacro:sick_laser_v0 name="lidar" parent="base_link_front_bumper_part" ros_topic="laser" update_rate="25" >
-    <origin xyz="0.03 0 0.05" rpy="0 0 0" />
+  <xacro:sick_laser_v0 name="lidar" parent="base_link_front_mount_part" ros_topic="laser" update_rate="25" >
+    <origin xyz="0.053086 0 -0.057912" rpy="0 0 0" />
   </xacro:sick_laser_v0>
   <gazebo reference="lidar">
@@ -40,5 +49,5 @@
   </gazebo>
   <!-- Arm -->
-  <xacro:static_transform parent="base_link_front_bumper_part" name="arm_base" xyz="-0.04 0 -0.03" rpy="0 0 0">
+  <xacro:static_transform parent="base_link_top_plate_part" name="arm_base" xyz="0.325374 0 0.085852" rpy="0 0 0">
     <visual>
       <origin xyz="0 0 0" rpy="0 0 0" />
@@ -50,5 +59,23 @@
   </xacro:static_transform>
   <!-- IMU -->
-  <xacro:static_transform parent="base_link" name="imu" xyz="0.06 0 0" rpy="0 0 0">
+  <xacro:static_transform parent="base_link" name="imu" xyz="0 0 0" rpy="0 0 0">
+    <visual>
+      <origin xyz="0 0 0" rpy="0 0 0" />
+      <geometry>
+	<box size="0.01 0.01 0.01" />
+      </geometry>
+      <material name="Blue" />
+    </visual>
+  </xacro:static_transform>
+  <xacro:static_transform parent="imu" name="imu/accel" xyz="0 0 0" rpy="0 0 0">
+    <visual>
+      <origin xyz="0 0 0" rpy="0 0 0" />
+      <geometry>
+	<box size="0.01 0.01 0.01" />
+      </geometry>
+      <material name="Blue" />
+    </visual>
+  </xacro:static_transform>
+  <xacro:static_transform parent="imu" name="imu/gyro" xyz="0 0 0" rpy="0 0 0">
     <visual>
       <origin xyz="0 0 0" rpy="0 0 0" />

File: aero_description/urdf/husky.urdf.xacro (robot description, xacro)
@@ -131,33 +131,16 @@
     <husky_wheel fb="front" lr="right" parent="base_link" translateX="1" translateY="-1" flipY="-1"/>
     <!-- DECORATIONS -->
-    <!-- Top Plate -->
     <husky_part parent="base_link" name="top_plate" mesh="top_plate"
 		colour="Yellow"
-		translateX="0.0" translateY="0.0" translateZ="0.005"
+		translateX="0.0" translateY="0.0" translateZ="0.2276"
 		rotateX="0.0" rotateY="0.0" rotateZ="0.0"/>
     <gazebo reference="base_link_top_plate_part">
       <material>Gazebo/Yellow</material>
     </gazebo>
-    <!-- User Rail -->
-    <husky_part parent="base_link" name="user_rail" mesh="user_rail"
+    <husky_part parent="base_link" name="front_mount" mesh="front_mount"
 		colour="DarkGray"
-		translateX="0.272" translateY="0.0" translateZ="0.245"
+		translateX="0.417068" translateY="0.0" translateZ="0.091"
 		rotateX="0.0" rotateY="0.0" rotateZ="0.0"/>
-    <gazebo reference="base_link_user_rail_part">
-      <material>Gazebo/Grey</material>
-    </gazebo>
-    <!-- Bumpers -->
-    <husky_part parent="base_link" name="front_bumper" mesh="bumper"
-		colour="DarkGray"
-		translateX="0.490" translateY="0.0" translateZ="0.091"
-		rotateX="0.0" rotateY="0.0" rotateZ="0.0"/>
-    <gazebo reference="base_link_front_bumper_part">
-      <material>Gazebo/FlatBlack</material>
-    </gazebo>
-    <husky_part parent="base_link" name="rear_bumper" mesh="bumper"
-		colour="DarkGray"
-		translateX="-0.48" translateY="0.0" translateZ="0.091"
-		rotateX="0.0" rotateY="0.0" rotateZ="3.14"/>
-    <gazebo reference="base_link_rear_bumper_part">
+    <gazebo reference="base_link_front_mount_part">
       <material>Gazebo/FlatBlack</material>
     </gazebo>

Commit message: Many many small bug fixes. Robot now correctly processes LIDAR data and can display it in rviz

File: aero_description/urdf/aero.urdf.xacro (robot description, xacro)
@@ -42,6 +42,6 @@
   </xacro:revolute_pan_transform>
   <!-- Laser -->
-  <xacro:sick_laser_v0 name="lidar" parent="base_link_front_mount_part" ros_topic="laser" update_rate="25" >
-    <origin xyz="0.053086 0 -0.057912" rpy="0 0 0" />
+  <xacro:sick_laser_v0 name="laser" parent="base_link_front_mount_part" ros_topic="laser" update_rate="25" >
+    <origin xyz="0.053086 0 -0.057912" rpy="${M_PI} 0 0" />
   </xacro:sick_laser_v0>
   <gazebo reference="lidar">

Commit message: Fixed wheel odometry covariances so that robot pose ekf will accept them

File: aero_description/urdf/aero.urdf.xacro (robot description, xacro)
@@ -68,21 +68,3 @@
     </visual>
   </xacro:static_transform>
-  <xacro:static_transform parent="imu" name="imu/accel" xyz="0 0 0" rpy="0 0 0">
-    <visual>
-      <origin xyz="0 0 0" rpy="0 0 0" />
-      <geometry>
-	<box size="0.01 0.01 0.01" />
-      </geometry>
-      <material name="Blue" />
-    </visual>
-  </xacro:static_transform>
-  <xacro:static_transform parent="imu" name="imu/gyro" xyz="0 0 0" rpy="0 0 0">
-    <visual>
-      <origin xyz="0 0 0" rpy="0 0 0" />
-      <geometry>
-	<box size="0.01 0.01 0.01" />
-      </geometry>
-      <material name="Blue" />
-    </visual>
-  </xacro:static_transform>
 </robot>

Commit message: cleaned up folders

File: aero_description/urdf/aero.urdf.xacro (robot description, xacro)
@@ -49,5 +49,14 @@
   </gazebo>
   <!-- Arm -->
-  <xacro:static_transform parent="base_link_top_plate_part" name="arm_base" xyz="0.325374 0 0.085852" rpy="0 0 ${-M_PI/2}">
+  <xacro:static_transform parent="base_link_top_plate_part" name="arm_mount" xyz="0.325374 0 0.085852" rpy="0 0 0">
+    <visual>
+      <origin xyz="0 0 0" rpy="0 0 0" />
+      <geometry>
+	<box size="0.01 0.01 0.01" />
+      </geometry>
+      <material name="Blue" />
+    </visual>
+  </xacro:static_transform>
+  <xacro:static_transform parent="arm_mount" name="arm_base" xyz="0 0 0" rpy="0 0 ${-M_PI/2}">
     <visual>
       <origin xyz="0 0 0" rpy="0 0 0" />

Commit message: Updated robot model with new boom and better measurements

File: aero_description/urdf/aero.urdf.xacro (robot description, xacro)
@@ -19,35 +19,43 @@
   <include filename="$(find aero_description)/urdf/sick_laser.urdf.xacro" />
   <include filename="$(find aero_description)/urdf/simple_transform.urdf.xacro" />
+  <property name="boom_length" value="1.0" />
+  <property name="boom_diameter" value="0.06" />
   <xacro:husky/>
-  <!-- Cameras -->
-  <xacro:stereo_camera_pair parent="base_link_front_mount_part" prefix="lower_stereo" xyz="0.07 0 0.02" rpy="0 ${M_PI/180*6} 0" camera_offset="0.08"/>
-  <xacro:stereo_camera_pair parent="boom" prefix="upper_stereo" xyz="0 0 0.022606" rpy="0 0 0" camera_offset="0.294386"/>
-  <xacro:static_transform parent="base_link_top_plate_part" name="boom_base" xyz="-0.422402 0 -0.09906" rpy="0 0 0">
+  <!-- Boom -->
+  <xacro:static_transform parent="top_plate" name="boom_base" xyz="-0.6 0 -0.09906" rpy="0 0 0">
     <visual>
-      <origin xyz="0 0 0" rpy="0 0 0" />
+      <origin xyz="0 0 -0.02" rpy="0 0 0" />
       <geometry>
-	<box size="0.01 0.01 0.01" />
+	<box size="0.04 0.04 0.04" />
       </geometry>
       <material name="Blue" />
     </visual>
   </xacro:static_transform>
-  <xacro:revolute_pan_transform parent="boom_base" name="boom" xyz="0 0 1.014476" rpy="0 0 0" lower_limit="-2" upper_limit="2">
+  <xacro:revolute_pan_transform parent="boom_base" name="boom" xyz="0 0 0" rpy="0 0 0" lower_limit="-2" upper_limit="2">
     <visual>
-      <origin xyz="0.0 0.0 -0.45" rpy="0 0 0" />
+      <origin xyz="0.0 0.0 ${boom_length/2}" rpy="0 0 0" />
       <geometry>
-	<cylinder length="0.9" radius="0.02" />
+	<cylinder length="${boom_length}" radius="${boom_diameter/2}" />
       </geometry>
-      <material name="DarkGray" />
+      <material name="Black" />
     </visual>
   </xacro:revolute_pan_transform>
+  <xacro:static_transform parent="boom" name="boom_top" xyz="0 0 ${boom_length}" rpy="0 0 0">
+    <visual>
+      <origin xyz="0 0 0" rpy="0 0 0" />
+      <geometry>
+	<box size="0.00 0.00 0.00" />
+      </geometry>
+    </visual>
+  </xacro:static_transform>
+  <!-- Cameras -->
+  <xacro:stereo_camera_pair parent="boom_top" prefix="upper_stereo" xyz="0 0 0.01" rpy="0 0 0" camera_base_length="0.3" camera_tilt="${10*M_PI/180}"/>
+  <xacro:stereo_camera_pair parent="boom_top" prefix="lower_stereo" xyz="0 0 -0.14" rpy="0 0 0" camera_base_length="0.11" camera_tilt="${30*M_PI/180}"/>
   <!-- Laser -->
-  <xacro:sick_laser_v0 name="laser" parent="base_link_front_mount_part" ros_topic="laser" update_rate="25" >
-    <origin xyz="0.053086 0 -0.057912" rpy="${M_PI} 0 0" />
+  <xacro:sick_laser_v0 name="laser" parent="base_link" ros_topic="laser" update_rate="25" >
+    <origin xyz="${base_length/2+0.0635} 0 0.0254" rpy="0 0 0" />
   </xacro:sick_laser_v0>
-  <gazebo reference="lidar">
-    <material>Gazebo/White</material>
-  </gazebo>
   <!-- Arm -->
-  <xacro:static_transform parent="base_link_top_plate_part" name="arm_mount" xyz="0.325374 0 0.085852" rpy="0 0 0">
+  <xacro:static_transform parent="base_link" name="arm_mount" xyz="0.325374 0 0.285852" rpy="0 0 0">
     <visual>
       <origin xyz="0 0 0" rpy="0 0 0" />

File: aero_description/urdf/husky.urdf.xacro (robot description, xacro)
@@ -40,40 +40,62 @@
     xmlns:physics="http://playerstage.sourceforge.net/gazebo/xmlschema/#physics"
 	xmlns:xacro="http://ros.org/wiki/xacro" name="aero">
-  <!-- Included URDF/XACRO Files -->
-  <include filename="$(find husky_description)/urdf/materials.urdf.xacro" />
-  <include filename="$(find aero_description)/urdf/wheel.urdf.xacro" />
-  <include filename="$(find aero_description)/urdf/parts.urdf.xacro" />
+  <!-- Colors -->
+  <material name="Black">
+    <color rgba="0.0 0.0 0.0 1.0"/>
+  </material>
+  <material name="Blue">
+    <color rgba="0.0 0.0 0.8 1.0"/>
+  </material>
+  <material name="Green">
+    <color rgba="0.0 0.8 0.0 1.0"/>
+  </material>
+  <material name="Gray">
+    <color rgba="0.7 0.7 0.7 1.0"/>
+  </material>
+  <material name="DarkGray">
+    <color rgba="0.3 0.3 0.3 1.0"/>
+  </material>
+  <material name="Red">
+    <color rgba="0.8 0.0 0.0 1.0"/>
+  </material>
+  <material name="White">
+    <color rgba="1.0 1.0 1.0 1.0"/>
+  </material>
+  <material name="Yellow">
+    <color rgba="0.8 0.8 0.0 1.0"/>
+  </material>
   <!-- PROPERTY LIST -->
   <!--All units in m-kg-s-radians unit system -->
   <property name="M_PI" value="3.1415926535897931" />
-  <!-- Main Body-base-->
-  <!-- Location of com : center of mass -->
-  <property name="base_x_com" value="-0.08748000" />
-  <property name="base_y_com" value="-0.00085000" />
-  <property name="base_z_com" value="0.09947000" />
-  <!-- Size of the base-->
-  <property name="base_x_size" value="0.98740000" />
-  <property name="base_y_size" value="0.57090000" />
-  <property name="base_z_size" value="0.24750000" />
-  <!--Weight of the base-->
-  <property name="base_mass" value="33.45489000" /> <!-- in kg-->
-  <!--Inertial values for the base at center of mass, aligned with coordinate system. Units are kg*m^2-->
-  <property name="base_ixx_com_cs" value="0.60216370" />
-  <property name="base_ixy_com_cs" value="-0.02364198" />
-  <property name="base_ixz_com_cs" value="-0.11972132" />
-  <property name="base_iyy_com_cs" value="1.73859574" />
-  <property name="base_iyz_com_cs" value="-0.00154437" />
-  <property name="base_izz_com_cs" value="2.02955229" />
+  <property name="base_length" value="0.806" />
+  <property name="base_width" value="0.419" />
+  <property name="base_height" value="0.228" />
+  <property name="wheel_diameter" value="0.32" />
+  <property name="wheel_width" value="0.11" />
+  <property name="wheel_base_width" value="0.546" />
+  <property name="wheel_base_length" value="0.558" />
+  <property name="wheel_base_link_height" value="0.0381" />
+  <property name="top_plate_length" value="0.549" />
+  <xacro:macro name="husky_wheel" params="fb lr parent translateX translateY flipY"> <!--fb : front, back ; lr: left, right -->
+    <link name="${fb}_${lr}_wheel">
+      <visual>
+	<origin xyz="0 0 0" rpy="${flipY*M_PI + M_PI/2} 0 0" />
+	<geometry>
+	  <cylinder radius="${wheel_diameter/2}" length="${wheel_width}" />
+	</geometry>
+	<material name="DarkGray" />
+      </visual>
+    </link>
+    <joint name="joint_${fb}_${lr}_wheel" type="continuous">
+      <parent link="${parent}"/>
+      <child link="${fb}_${lr}_wheel"/>
+      <origin xyz="${translateX * wheel_base_length/2} ${translateY * wheel_base_width/2} ${wheel_base_link_height}" rpy="0 0 0" />
+      <axis xyz="0 1 0" rpy="0 0 0" />
+      <limit effort="100" velocity="100"/>
+      <joint_properties damping="0.0" friction="0.0"/>
+    </joint>
+  </xacro:macro>
   <xacro:macro name="husky">
-    <!-- BASE-FOOTPRINT -->
-    <!-- base_footprint is a fictitious link(frame) that is on the ground right below base_link origin, navigation stack depends on this frame -->
     <link name="base_footprint">
-      <inertial>
-	<mass value="0.0001" />
-	<origin xyz="0 0 0" />
-	<inertia ixx="0.0001" ixy="0.0" ixz="0.0"
-		 iyy="0.0001" iyz="0.0"
-		 izz="0.0001" />
-      </inertial>
       <visual>
 	<origin xyz="0 0 0" rpy="0 0 0" />
@@ -81,48 +103,25 @@
 	  <box size="0.001 0.001 0.001" />
 	</geometry>
+	<material name="Blue" />
       </visual>
     </link>
-    <gazebo reference="base_footprint">
-      <material>Gazebo/Green</material>
-      <turnGravityOff>false</turnGravityOff>
-    </gazebo>
-    <joint name="base_link_joint" type="fixed">
-      <origin xyz="0 0 ${wheel_x_size/2 - base_z_origin_to_wheel_origin - base_z_origin_offset - base_z_origin_offset}" rpy="0 0 0" />
-      <parent link="base_footprint"/>
-      <child link="base_link" />
-    </joint>
-    <!-- BASE-LINK -->
-    <!--Actual body/chassis of the robot-->
-    <link name="base_link">
-      <inertial>
-	<mass value="${base_mass}" />
-	<!--This is the pose of the inertial reference frame, relative to the link reference frame. The origin of the inertial reference frame needs to be at the center of gravity. The axes of the inertial reference frame do not need to be aligned with the principal axes of the inertia.-->
-	<origin xyz="${base_x_com} ${base_y_com} ${base_z_com}" />
-	<!--The 3x3 rotational inertia matrix. Because the rotational inertia matrix is symmetric, only 6 above-diagonal elements of this matrix are specified here, using the attributes ixx, ixy, ixz, iyy, iyz, izz.-->
-	<inertia ixx="${base_ixx_com_cs}" ixy="${base_ixy_com_cs}" ixz="${base_ixz_com_cs}"
-		 iyy="${base_iyy_com_cs}" iyz="${base_iyz_com_cs}" izz="${base_izz_com_cs}" />
-      </inertial>
-      <visual>
-<!--	<origin xyz="0 0 ${base_z_origin_offset}" rpy="0 0 0" />
-	<geometry>
-	  <mesh filename="package://husky_description/Media/models/base_link.stl" />
-	</geometry>-->
-	<origin xyz="0 0 ${wheel_x_size/2 - base_z_origin_to_wheel_origin - 0.02}" rpy="0 0 0 " />
-	<geometry>
-	  <box size = "${base_x_size+0.02} ${base_y_size} ${base_z_size + 0.02}"/> <!--making it slightly bigger in x and z direction-->
-	</geometry>
-	<material name="Black" />
-      </visual>
-      <collision>
-	<origin xyz="0 0 ${wheel_x_size/2 - base_z_origin_to_wheel_origin - 0.02}" rpy="0 0 0 " />
-	<geometry>
-	  <box size = "${base_x_size+0.02} ${base_y_size} ${base_z_size + 0.02}"/> <!--making it slightly bigger in x and z direction-->
-	</geometry>
-      </collision>
-    </link>
-    <gazebo reference="base_link">
-      <material>Gazebo/FlatBlack</material>
-      <turnGravityOff>false</turnGravityOff>
-    </gazebo>
+  <xacro:static_transform parent="base_footprint" name="base_link" xyz="0 0 ${wheel_diameter/2-wheel_base_link_height}" rpy="0 0 0">
+    <visual>
+      <origin xyz="0 0 ${base_height/2}" rpy="0 0 0" />
+      <geometry>
+	<box size="${base_length} ${base_width} ${base_height}" />
+      </geometry>
+      <material name="Yellow" />
+    </visual>
+  </xacro:static_transform>
+  <xacro:static_transform parent="base_link" name="top_plate" xyz="0 0 ${base_height}" rpy="0 0 0">
+    <visual>
+      <origin xyz="0 0 0" rpy="0 0 0" />
+      <geometry>
+	<box size="${top_plate_length} ${base_width} 0.02" />
+      </geometry>
+      <material name="DarkGray" />
+    </visual>
+  </xacro:static_transform>
     <!-- WHEEL macros -->
     <husky_wheel fb="back" lr="left" parent="base_link" translateX="-1" translateY="1" flipY="-1"/>
@@ -130,32 +129,4 @@
     <husky_wheel fb="front" lr="left" parent="base_link" translateX="1" translateY="1" flipY="-1"/>
     <husky_wheel fb="front" lr="right" parent="base_link" translateX="1" translateY="-1" flipY="-1"/>
-    <!-- DECORATIONS -->
-    <husky_part parent="base_link" name="top_plate" mesh="top_plate"
-		colour="Yellow"
-		translateX="0.0" translateY="0.0" translateZ="0.2276"
-		rotateX="0.0" rotateY="0.0" rotateZ="0.0"/>
-    <gazebo reference="base_link_top_plate_part">
-      <material>Gazebo/Yellow</material>
-    </gazebo>
-    <husky_part parent="base_link" name="front_mount" mesh="front_mount"
-		colour="DarkGray"
-		translateX="0.417068" translateY="0.0" translateZ="0.091"
-		rotateX="0.0" rotateY="0.0" rotateZ="0.0"/>
-    <gazebo reference="base_link_front_mount_part">
-      <material>Gazebo/FlatBlack</material>
-    </gazebo>
-    <gazebo>
-      <controller:husky_plugin name="husky_diff_controller" plugin="libhusky_description.so">
-	<alwaysOn>true</alwaysOn>
-	<updateRate>100.0</updateRate>
-	<backLeftJoint>joint_back_left_wheel</backLeftJoint>
-	<backRightJoint>joint_back_right_wheel</backRightJoint>
-	<frontLeftJoint>joint_front_left_wheel</frontLeftJoint>
-	<frontRightJoint>joint_front_right_wheel</frontRightJoint>
-	<wheelSeparation>${base_y_size}</wheelSeparation>
-	<wheelDiameter>${wheel_x_size}</wheelDiameter>
-	<torque>35</torque>
-      </controller:husky_plugin>
-    </gazebo>
   </xacro:macro>
 </root>

File: aero_description/urdf/manta_camera.urdf.xacro (robot description, xacro)
@@ -5,4 +5,6 @@
       xmlns:xacro="http://ros.org/wiki/xacro">
   <include filename="$(find aero_description)/urdf/manta_camera.gazebo.xacro" />
+  <property name="manta_camera_width" value="0.04" />
+  <property name="manta_camera_height" value="0.02" />
   <xacro:macro name="manta_cam_v0" params="frame_name parent *origin camera_name">
     <joint name="${frame_name}_frame_joint" type="fixed">

File: aero_description/urdf/stereo_camera_pair.urdf.xacro (robot description, xacro)
@@ -6,19 +6,21 @@
   <include filename="$(find aero_description)/urdf/simple_transform.urdf.xacro" />
   <include filename="$(find aero_description)/urdf/manta_camera.urdf.xacro" />
-  <xacro:macro name="stereo_camera_pair" params="prefix parent xyz rpy camera_offset">
+  <property name="camera_rail_length" value="0.04" /><!--front to back -->
+  <property name="camera_rail_height" value="0.02" />
+  <xacro:macro name="stereo_camera_pair" params="prefix parent xyz rpy camera_base_length camera_tilt">
     <xacro:static_transform parent="${parent}" name="${prefix}/camera_rail" xyz="${xyz}" rpy="${rpy}">
     <visual>
-      <origin xyz="-0.03 0 -0.018" rpy="0 0 0" />
+      <origin xyz="0 0 0" rpy="0 0 0" />
       <geometry>
-	<box size="0.05 ${camera_offset+0.04} 0.013" />
+	<box size="${camera_rail_length} ${camera_base_length-manta_camera_width} ${camera_rail_height}" />
       </geometry>
-      <material name="Red"/>
+      <material name="Blue"/>
     </visual>
   </xacro:static_transform>
     <xacro:manta_cam_v0 frame_name="${prefix}/left_camera" parent="${prefix}/camera_rail" camera_name="${prefix}/left">
-      <origin xyz="0.0 ${camera_offset/2} 0.0" rpy="0 0 0" />
+      <origin xyz="0.03 ${camera_base_length/2} ${manta_camera_height/2+camera_rail_height/2}" rpy="0 ${camera_tilt} 0" />
     </xacro:manta_cam_v0>
     <xacro:manta_cam_v0 frame_name="${prefix}/right_camera" parent="${prefix}/camera_rail" camera_name="${prefix}/right">
-      <origin xyz="0.0 ${-camera_offset/2} 0.0" rpy="0 0 0" />
+      <origin xyz="0.03 ${-camera_base_length/2} ${manta_camera_height/2+camera_rail_height/2}" rpy="0 ${camera_tilt} 0" />
     </xacro:manta_cam_v0>
     <xacro:static_transform parent="${prefix}/camera_rail" name="${prefix}_optical_frame" xyz="0 0 0" rpy="${-M_PI/2} 0 ${-M_PI/2}">
