Commit message: Updated robot model

File: aero_description/urdf/aero.urdf.xacro (robot description, xacro)
@@ -19,9 +19,11 @@
   <include filename="$(find aero_description)/urdf/sick_laser.urdf.xacro" />
   <include filename="$(find aero_description)/urdf/simple_transform.urdf.xacro" />
-  <property name="boom_length" value="1.0" />
-  <property name="boom_diameter" value="0.06" />
+  <include filename="$(find aero_description)/urdf/simple_transform.urdf.xacro" />
+  <include filename="$(find jaco_model)/urdf/jaco_arm.xacro" />
+  <property name="boom_length" value="1.085" />
+  <property name="boom_diameter" value="0.0538" />
   <xacro:husky/>
   <!-- Boom -->
-  <xacro:static_transform parent="top_plate" name="boom_base" xyz="-0.6 0 -0.09906" rpy="0 0 0">
+  <xacro:static_transform parent="top_plate" name="boom_base" xyz="-0.2 0 0.0762" rpy="0 0 0">
     <visual>
       <origin xyz="0 0 -0.02" rpy="0 0 0" />
@@ -50,6 +52,6 @@
   </xacro:static_transform>
   <!-- Cameras -->
-  <xacro:stereo_camera_pair parent="boom_top" prefix="upper_stereo" xyz="0 0 0.01" rpy="0 0 0" camera_base_length="0.3" camera_tilt="${10*M_PI/180}"/>
-  <xacro:stereo_camera_pair parent="boom_top" prefix="lower_stereo" xyz="0 0 -0.14" rpy="0 0 0" camera_base_length="0.11" camera_tilt="${30*M_PI/180}"/>
+  <xacro:stereo_camera_pair parent="boom_top" prefix="upper_stereo" xyz="0 0 0.005" rpy="0 0 0" camera_base_length="0.3" camera_tilt="${10*M_PI/180}"/>
+  <xacro:stereo_camera_pair parent="boom_top" prefix="lower_stereo" xyz="0 0 -0.127" rpy="0 0 0" camera_base_length="0.11" camera_tilt="${30*M_PI/180}"/>
   <!-- Laser -->
   <xacro:sick_laser_v0 name="laser" parent="base_link" ros_topic="laser" update_rate="25" >
@@ -57,5 +59,5 @@
   </xacro:sick_laser_v0>
   <!-- Arm -->
-  <xacro:static_transform parent="base_link" name="arm_mount" xyz="0.325374 0 0.285852" rpy="0 0 0">
+  <xacro:static_transform parent="base_link" name="arm_mount" xyz="0.325374 0 0.1" rpy="0 0 0">
     <visual>
       <origin xyz="0 0 0" rpy="0 0 0" />
@@ -75,4 +77,5 @@
     </visual>
   </xacro:static_transform>
+<xacro:jaco_arm  parent="arm_base"/>
   <!-- IMU -->
   <xacro:static_transform parent="base_link" name="imu" xyz="0 0 0" rpy="0 ${-M_PI/2} ${-3*M_PI/4}">

File: aero_description/urdf/stereo_camera_pair.urdf.xacro (robot description, xacro)
@@ -6,10 +6,10 @@
   <include filename="$(find aero_description)/urdf/simple_transform.urdf.xacro" />
   <include filename="$(find aero_description)/urdf/manta_camera.urdf.xacro" />
-  <property name="camera_rail_length" value="0.04" /><!--front to back -->
-  <property name="camera_rail_height" value="0.02" />
+  <property name="camera_rail_length" value="0.0508" /><!--front to back -->
+  <property name="camera_rail_height" value="0.0254" />
   <xacro:macro name="stereo_camera_pair" params="prefix parent xyz rpy camera_base_length camera_tilt">
     <xacro:static_transform parent="${parent}" name="${prefix}/camera_rail" xyz="${xyz}" rpy="${rpy}">
     <visual>
-      <origin xyz="0 0 0" rpy="0 0 0" />
+      <origin xyz="0 0 ${camera_rail_height/2}" rpy="0 0 0" />
       <geometry>
 	<box size="${camera_rail_length} ${camera_base_length-manta_camera_width} ${camera_rail_height}" />
@@ -18,11 +18,19 @@
     </visual>
   </xacro:static_transform>
-    <xacro:manta_cam_v0 frame_name="${prefix}/left_camera" parent="${prefix}/camera_rail" camera_name="${prefix}/left">
-      <origin xyz="0.03 ${camera_base_length/2} ${manta_camera_height/2+camera_rail_height/2}" rpy="0 ${camera_tilt} 0" />
+  <xacro:static_transform parent="${prefix}/camera_rail" name="${prefix}/camera_rail_tilt" xyz="0 0 ${camera_rail_height/2}" rpy="0 ${camera_tilt} 0">
+    <visual>
+      <origin xyz="0 0 0" rpy="0 0 0" />
+      <geometry>
+	<box size="0 0 0" />
+      </geometry>
+    </visual>
+  </xacro:static_transform>
+    <xacro:manta_cam_v0 frame_name="${prefix}/left_camera" parent="${prefix}/camera_rail_tilt" camera_name="${prefix}/left">
+      <origin xyz="0.03 ${camera_base_length/2} ${manta_camera_height/2+camera_rail_height/2}" rpy="0 0 0" />
     </xacro:manta_cam_v0>
-    <xacro:manta_cam_v0 frame_name="${prefix}/right_camera" parent="${prefix}/camera_rail" camera_name="${prefix}/right">
-      <origin xyz="0.03 ${-camera_base_length/2} ${manta_camera_height/2+camera_rail_height/2}" rpy="0 ${camera_tilt} 0" />
+    <xacro:manta_cam_v0 frame_name="${prefix}/right_camera" parent="${prefix}/camera_rail_tilt" camera_name="${prefix}/right">
+      <origin xyz="0.03 ${-camera_base_length/2} ${manta_camera_height/2+camera_rail_height/2}" rpy="0 0 0" />
     </xacro:manta_cam_v0>
-    <xacro:static_transform parent="${prefix}/camera_rail" name="${prefix}_optical_frame" xyz="0 0 0" rpy="${-M_PI/2} 0 ${-M_PI/2}">
+    <xacro:static_transform parent="${prefix}/camera_rail_tilt" name="${prefix}_optical_frame" xyz="0.03 0 ${manta_camera_height/2+camera_rail_height/2}" rpy="${-M_PI/2} 0 ${-M_PI/2}">
     <visual>
       <geometry>

Commit message: Updated robot model to reflect temporary boom mount

File: aero_description/urdf/aero.urdf.xacro (robot description, xacro)
@@ -25,9 +25,9 @@
   <xacro:husky/>
   <!-- Boom -->
-  <xacro:static_transform parent="top_plate" name="boom_base" xyz="-0.2 0 0.0762" rpy="0 0 0">
+  <xacro:static_transform parent="top_plate" name="boom_base" xyz="-0.23 0 0.0762" rpy="0 0 0">
     <visual>
       <origin xyz="0 0 -0.02" rpy="0 0 0" />
       <geometry>
-	<box size="0.04 0.04 0.04" />
+	<box size="0.05 0.05 0.05" />
       </geometry>
       <material name="Blue" />

Commit message: Changes from outside testing

File: aero_description/urdf/aero.urdf.xacro (robot description, xacro)
@@ -56,5 +56,5 @@
   <!-- Laser -->
   <xacro:sick_laser_v0 name="laser" parent="base_link" ros_topic="laser" update_rate="25" >
-    <origin xyz="${base_length/2+0.0635} 0 0.0254" rpy="0 0 0" />
+    <origin xyz="${base_length/2+0.0635} 0 0.0254" rpy="${M_PI} 0 0" />
   </xacro:sick_laser_v0>
   <!-- Arm -->

Commit message: Modifications to account for the now non-inverted laser. closes #118

File: aero_description/urdf/aero.urdf.xacro (robot description, xacro)
@@ -56,5 +56,5 @@
   <!-- Laser -->
   <xacro:sick_laser_v0 name="laser" parent="base_link" ros_topic="laser" update_rate="25" >
-    <origin xyz="${base_length/2+0.0635} 0 0.0254" rpy="${M_PI} 0 0" />
+    <origin xyz="${base_length/2+0.0635} 0 0.0254" rpy="0 0 0" />
   </xacro:sick_laser_v0>
   <!-- Arm -->
